File: FPV-Treff - Groundstation.brd (EAGLE design)
At the start: 67 x 61 mm, 37 parts, among them IC1 TINY13-20PU, J1 XT-60BATT_LABEL, Q1 BC337, Q2 BC337, Q3 BC337, Q4 BC337, Q5 BS170T

Commit message: Add files via upload
Parts:
- added R11: 75R, resistor:0204V
- JP3: value (none) -> Goggles
- moved C5 5.71 mm to (22.9, 53.3)
- moved L1 3.70 mm to (1.27, 28.6)
- moved JP3 2.54 mm to (4.45, 23.5)
Connections:
- net GND: now also R11.1
- net N$2: now also C6.+, JP1.1, L1.2; no longer C5.-, VIDEO_IN.1
- net N$5: now also C7.+
- net N$7: no longer C6.+
- net N$8: now also C5.-, R11.2, VIDEO_IN.1; no longer JP1.1, L1.2
- net N$9: no longer C7.+
Routing:
- net N$8: track 9.04 -> 21.1 mm
- net N$56: track 94.9 -> 89.1 mm
- net N$9: track 11.7 -> 6.43 mm
- net N$5: track 62.2 -> 66.0 mm
- net N$2: track 12.8 -> 16.5 mm
- net N$7: track 65.8 -> 67.3 mm
- net GND: vias 1 -> 3

Commit message: Add files via upload
Parts:
- removed D1: 5,1V, diode:ZDIO-5
- removed Q5: BS170T, gm-trans:SOT54E
- removed R10: 100, rcl:0207/10
- removed R8: 4k7, rcl:0207/10
- removed R9: 15, rcl:0207/10
- added C9: 100nF, rcl:C025_050-025X075
- added IC2: 7805L, adafruit2:TO92
- JP1: value (none) -> Goggles
- JP3: value Goggles -> 5V_Piezo
- moved C8 6.84 mm to (15.2, 27.3)
- moved L1 1.27 mm to (2.54, 28.6)
Connections:
- removed net N$13: C8.1, D1.C, IC1.8, R8.1
- removed net N$16: JP3.2, R10.2, R9.2
- net GND: now also C9.2, IC2.2, JP3.2; no longer D1.A, Q5.S, R10.1
- net N$11: now also JP3.1; no longer Q5.D, R9.1
- net N$12: now also C9.1, IC1.8, IC2.1; no longer IC1.6, Q5.G
- net N$7: now also C8.1, IC2.3; no longer JP3.1, R8.2
Routing:
- net N$16: track 16.1 -> 0.00 mm
- net N$7: track 67.3 -> 81.1 mm
- net N$13: track 13.8 -> 0.00 mm
- net N$12: track 14.9 -> 23.3 mm
- net N$11: track 6.93 -> 0.00 mm
