File: FPV-Treff - Groundstation.sch (EAGLE design)
At the start: 37 parts, among them IC1 TINY13-20PU, J1 XT-60BATT_LABEL, Q1 BC337, Q2 BC337, Q3 BC337, Q4 BC337, Q5 BS170T

Commit message: Add files via upload
Parts:
- added R11: 75R, resistor:R-EU_0204/2V
- JP3: value (none) -> Goggles
Connections:
- net GND: now also R11.1
- net N$2: now also C6.+, JP1.1, L1.2; no longer C5.-, VIDEO_IN.1
- net N$5: now also C7.+
- net N$7: no longer C6.+
- net N$8: now also C5.-, R11.2, VIDEO_IN.1; no longer JP1.1, L1.2
- net N$9: no longer C7.+
Other:
- moved on the sheet: C6, C7, JP1, L1, L2
Changed lines of the file:
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@@
 <part name="IC1" library="atmel(1)" deviceset="TINY13" device="PU" technology="-20"/>
 <part name="JP2" library="pinhead-1" deviceset="PINHD-1X2" device="_2.54"/>
-<part name="JP3" library="pinhead-1" deviceset="PINHD-1X2" device="_2.54"/>
+<part name="JP3" library="pinhead-1" deviceset="PINHD-1X2" device="_2.54" value="Goggles"/>
 <part name="R6" library="rcl" deviceset="R-EU_" device="0207/10" value="68k"/>
 <part name="R7" library="rcl" deviceset="R-EU_" device="0207/10" value="4k7"/>
@@
 <part name="GND17" library="supply1" deviceset="GND" device=""/>
 <part name="GND18" library="supply1" deviceset="GND" device=""/>
+<part name="R11" library="resistor" deviceset="R-EU_" device="0204/2V" value="75R"/>
+<part name="GND13" library="supply1" deviceset="GND" device=""/>
 </parts>
 <sheets>
@@
 <instance part="GND36" gate="1" x="261.62" y="144.78"/>
 <instance part="GND37" gate="1" x="261.62" y="228.6"/>
-<instance part="L1" gate="G$1" x="203.2" y="281.94" rot="R90"/>
+<instance part="L1" gate="G$1" x="195.58" y="281.94" rot="R90"/>
 <instance part="C5" gate="G$1" x="246.38" y="162.56" rot="R270"/>
 <instance part="C4" gate="G$1" x="279.4" y="157.48" rot="R90"/>
@@
 <instance part="GND6" gate="1" x="193.04" y="241.3"/>
 <instance part="U$1" gate="G$1" x="208.28" y="254"/>
-<instance part="C6" gate="G$1" x="195.58" y="274.32"/>
-<instance part="GND7" gate="1" x="195.58" y="264.16"/>
-<instance part="GND8" gate="1" x="208.28" y="264.16"/>
-<instance part="JP1" gate="A" x="218.44" y="279.4"/>
+<instance part="C6" gate="G$1" x="203.2" y="274.32"/>
+<instance part="GND7" gate="1" x="203.2" y="264.16"/>
+<instance part="GND8" gate="1" x="213.36" y="264.16"/>
+<instance part="JP1" gate="A" x="223.52" y="279.4"/>
 <instance part="GND9" gate="1" x="228.6" y="241.3"/>
-<instance part="L2" gate="G$1" x="241.3" y="256.54" rot="R90"/>
-<instance part="C7" gate="G$1" x="233.68" y="251.46"/>
-<instance part="GND10" gate="1" x="233.68" y="241.3"/>
+<instance part="L2" gate="G$1" x="233.68" y="256.54" rot="R90"/>
+<instance part="C7" gate="G$1" x="241.3" y="251.46"/>
+<instance part="GND10" gate="1" x="241.3" y="241.3"/>
 <instance part="Q5" gate="1" x="200.66" y="185.42"/>
 <instance part="IC1" gate="G$1" x="170.18" y="177.8"/>
@@
 <instance part="GND17" gate="1" x="203.2" y="175.26"/>
 <instance part="GND18" gate="1" x="210.82" y="175.26"/>
+<instance part="R11" gate="G$1" x="236.22" y="154.94" rot="R90"/>
+<instance part="GND13" gate="1" x="236.22" y="144.78"/>
 </instances>
 <busses>
@@
 <pinref part="C6" gate="G$1" pin="-"/>
 <pinref part="GND7" gate="1" pin="GND"/>
-<wire x1="195.58" y1="266.7" x2="195.58" y2="269.24" width="0.1524" layer="91"/>
+<wire x1="203.2" y1="266.7" x2="203.2" y2="269.24" width="0.1524" layer="91"/>
 </segment>
 <segment>
 <pinref part="JP1" gate="A" pin="3"/>
 <pinref part="GND8" gate="1" pin="GND"/>
-<wire x1="215.9" y1="276.86" x2="208.28" y2="276.86" width="0.1524" layer="91"/>
-<wire x1="208.28" y1="276.86" x2="208.28" y2="266.7" width="0.1524" layer="91"/>
+<wire x1="220.98" y1="276.86" x2="213.36" y2="276.86" width="0.1524" layer="91"/>
+<wire x1="213.36" y1="276.86" x2="213.36" y2="266.7" width="0.1524" layer="91"/>
 </segment>
 <segment>
@@
 <pinref part="C7" gate="G$1" pin="-"/>
 <pinref part="GND10" gate="1" pin="GND"/>
-<wire x1="233.68" y1="246.38" x2="233.68" y2="243.84" width="0.1524" layer="91"/>
+<wire x1="241.3" y1="246.38" x2="241.3" y2="243.84" width="0.1524" layer="91"/>
 </segment>
 <segment>
@@
 <pinref part="C8" gate="G$1" pin="2"/>
 <wire x1="147.32" y1="198.12" x2="147.32" y2="195.58" width="0.1524" layer="91"/>
+</segment>
+<segment>
+<pinref part="R11" gate="G$1" pin="1"/>
+<pinref part="GND13" gate="1" pin="GND"/>
+<wire x1="236.22" y1="147.32" x2="236.22" y2="149.86" width="0.1524" layer="91"/>
 </segment>
 </net>
@@
 </segment>
 </net>
-<net name="N$2" class="0">
-<segment>
-<pinref part="C5" gate="G$1" pin="-"/>
-<wire x1="241.3" y1="162.56" x2="223.52" y2="162.56" width="0.1524" layer="91"/>
-<pinref part="VIDEO_IN" gate="G$1" pin="1"/>
-</segment>
-</net>
 <net name="N$5" class="0">
 <segment>
-<pinref part="R5" gate="G$1" pin="2"/>
 <pinref part="Q1" gate="G$1" pin="C"/>
 <wire x1="261.62" y1="251.46" x2="269.24" y2="251.46" width="0.1524" layer="91"/>
 <wire x1="269.24" y1="251.46" x2="269.24" y2="256.54" width="0.1524" layer="91"/>
 <wire x1="269.24" y1="256.54" x2="251.46" y2="256.54" width="0.1524" layer="91"/>
+<wire x1="251.46" y1="256.54" x2="241.3" y2="256.54" width="0.1524" layer="91"/>
+<wire x1="241.3" y1="256.54" x2="238.76" y2="256.54" width="0.1524" layer="91"/>
 <wire x1="269.24" y1="251.46" x2="269.24" y2="223.52" width="0.1524" layer="91"/>
 <junction x="269.24" y="251.46"/>
@@
 <junction x="269.24" y="223.52"/>
 <pinref part="L2" gate="G$1" pin="2"/>
-<wire x1="246.38" y1="256.54" x2="251.46" y2="256.54" width="0.1524" layer="91"/>
+<pinref part="R5" gate="G$1" pin="2"/>
 <junction x="251.46" y="256.54"/>
+<pinref part="C7" gate="G$1" pin="+"/>
+<wire x1="241.3" y1="254" x2="241.3" y2="256.54" width="0.1524" layer="91"/>
+<junction x="241.3" y="256.54"/>
 </segment>
 </net>
@@
 <pinref part="U$1" gate="G$1" pin="VIN+"/>
 <wire x1="187.96" y1="256.54" x2="190.5" y2="256.54" width="0.1524" layer="91"/>
-<pinref part="L1" gate="G$1" pin="1"/>
 <wire x1="190.5" y1="256.54" x2="193.04" y2="256.54" width="0.1524" layer="91"/>
-<wire x1="198.12" y1="281.94" x2="195.58" y2="281.94" width="0.1524" layer="91"/>
-<wire x1="195.58" y1="281.94" x2="190.5" y2="281.94" width="0.1524" layer="91"/>
 <wire x1="190.5" y1="281.94" x2="190.5" y2="256.54" width="0.1524" layer="91"/>
 <junction x="190.5" y="256.54"/>
-<pinref part="C6" gate="G$1" pin="+"/>
-<wire x1="195.58" y1="276.86" x2="195.58" y2="281.94" width="0.1524" layer="91"/>
-<junction x="195.58" y="281.94"/>
 <pinref part="JP3" gate="G$1" pin="1"/>
 <pinref part="R6" gate="G$1" pin="2"/>
@@
 <wire x1="190.5" y1="256.54" x2="190.5" y2="220.98" width="0.1524" layer="91"/>
 <junction x="190.5" y="220.98"/>
-</segment>
-</net>
-<net name="N$8" class="0">
-<segment>
-<pinref part="L1" gate="G$1" pin="2"/>
-<pinref part="JP1" gate="A" pin="1"/>
-<wire x1="215.9" y1="281.94" x2="208.28" y2="281.94" width="0.1524" layer="91"/>
-</segment>
-</net>
-<net name="N$9" class="0">
-<segment>
-<pinref part="U$1" gate="G$1" pin="VOUT+"/>
-<pinref part="L2" gate="G$1" pin="1"/>
-<wire x1="226.06" y1="256.54" x2="233.68" y2="256.54" width="0.1524" layer="91"/>
-<pinref part="C7" gate="G$1" pin="+"/>
-<wire x1="233.68" y1="256.54" x2="236.22" y2="256.54" width="0.1524" layer="91"/>
-<wire x1="233.68" y1="254" x2="233.68" y2="256.54" width="0.1524" layer="91"/>
-<junction x="233.68" y="256.54"/>
+<pinref part="L1" gate="G$1" pin="1"/>
 </segment>
 </net>
@@
 </segment>
 </net>
+<net name="N$9" class="0">
+<segment>
+<pinref part="U$1" gate="G$1" pin="VOUT+"/>
+<pinref part="L2" gate="G$1" pin="1"/>
+<wire x1="228.6" y1="256.54" x2="226.06" y2="256.54" width="0.1524" layer="91"/>
+</segment>
+</net>
+<net name="N$2" class="0">
+<segment>
+<pinref part="JP1" gate="A" pin="1"/>
+<pinref part="L1" gate="G$1" pin="2"/>
+<wire x1="200.66" y1="281.94" x2="203.2" y2="281.94" width="0.1524" layer="91"/>
+<pinref part="C6" gate="G$1" pin="+"/>
+<wire x1="203.2" y1="281.94" x2="220.98" y2="281.94" width="0.1524" layer="91"/>
+<wire x1="203.2" y1="276.86" x2="203.2" y2="281.94" width="0.1524" layer="91"/>
+<junction x="203.2" y="281.94"/>
+</segment>
+</net>
+<net name="N$8" class="0">
+<segment>
+<pinref part="VIDEO_IN" gate="G$1" pin="1"/>
+<pinref part="C5" gate="G$1" pin="-"/>
+<wire x1="223.52" y1="162.56" x2="236.22" y2="162.56" width="0.1524" layer="91"/>
+<pinref part="R11" gate="G$1" pin="2"/>
+<wire x1="236.22" y1="162.56" x2="241.3" y2="162.56" width="0.1524" layer="91"/>
+<wire x1="236.22" y1="160.02" x2="236.22" y2="162.56" width="0.1524" layer="91"/>
+<junction x="236.22" y="162.56"/>
+</segment>
+</net>

Commit message: Add files via upload
Parts:
- removed D1: 5,1V, diode:ZENER-DIODEZD-5
- removed Q5: BS170T, gm-trans:BS170T
- removed R10: 100, rcl:R-EU_0207/10
- removed R8: 4k7, rcl:R-EU_0207/10
- removed R9: 15, rcl:R-EU_0207/10
- added C9: 100nF, rcl:C-EU025_050-025X075
- added IC2: 7805L, adafruit2:7805L
- JP1: value (none) -> Goggles
- JP3: value Goggles -> 5V_Piezo
Connections:
- removed net N$13: C8.1, D1.C, IC1.VCC, R8.1
- removed net N$16: JP3.2, R10.2, R9.2
- net GND: now also C9.2, IC2.GND, JP3.2; no longer D1.A, Q5.S, R10.1
- net N$11: now also JP3.1; no longer Q5.D, R9.1
- net N$12: now also C9.1, IC1.VCC, IC2.VO; no longer IC1.PB1/PCINT1/AIN1/OC0B/INT0/MISO, Q5.G
- net N$7: now also C8.1, IC2.VI; no longer JP3.1, R8.2
Other:
- moved on the sheet: C8, IC1, JP2, JP3, R7
